Commit message: second assignment

File: scripts/SECOND.urdf (robot description, URDF)
Before this commit: robot SECOND, 6 links, 5 joints
Links:
- added link LINKCAM
Joints:
- added joint JOINTCAM: type fixed, parent LINK4, child LINKCAM, origin xyz=0 0.03 0 rpy=0 0 1.5708

Commit message: add cam

File: scripts/SECOND.urdf (robot description, URDF)
Before this commit: robot SECOND, 7 links, 6 joints
Links:
- added link LINKCAMOPT
Joints:
- added joint JOINTCAMOPT: type fixed, parent LINKCAM, child LINKCAMOPT, origin xyz=0 0 0 rpy=-1.5708 0 -1.5708
